File: board/board.sch (KiCad schematic (older format))
At the start: 8 parts, among them U1 STM32F031K6, U2 AP2210

Commit message: create GPIO Pins
Parts:
- added C? (x3): 100nF, symbol Device:C
- added C?: 1nF, symbol Device:C
- added C?: 10nF, symbol Device:C
- added C? (x2): 20pF, symbol Device:C
- added FB?: Ferrite_Bead, symbol Device:Ferrite_Bead
- added J?: GPIO1, symbol Connector:Conn_01x12_Male
- added J?: GPIO2, symbol Connector:Conn_01x12_Male
- added J?: PROG, symbol Connector:Conn_01x04_Male
- added SW?: RESET, symbol Switch:SW_Push
- added Y?: 8MHz, symbol Device:Crystal
- R1: value 220R -> 4.7k
Connections:
- net +3V3: now also U1.1 (VDD), U1.17 (VDD), C?.1, C?.2, FB?.2, J?.11 (Pin_11)
- net GND: now also U1.16 (VSS), U1.31 (BOOT0), U1.32 (VSS), C?.1, C?.1, C?.1, C?.2, C?.2, C?.2, C?.2, J?.1 (Pin_1), J?.12 (Pin_12), SW?.2
- net VPP: now also J?.1 (Pin_1), J?.2 (Pin_2)
- net at U1.2 (XTO): now also C?.2, Y?.2
- net at U1.4 (NRST): now also C?.2, SW?.1
- net at U1.5 (VDDA): now also C?.1, C?.1, FB?.1
- new net: C?.1, U1.2 (XTO), Y?.1
- new net A0: J?.10 (Pin_10)
- new net A1: J?.9 (Pin_9)
- new net A10: J?.10 (Pin_10)
- new net A11: J?.9 (Pin_9)
- new net A12: J?.8 (Pin_8)
- new net A15: J?.7 (Pin_7)
- new net A2: J?.8 (Pin_8)
- new net A3: J?.7 (Pin_7)
- new net A4: J?.6 (Pin_6)
- new net A5: J?.5 (Pin_5)
- new net A6: J?.4 (Pin_4)
- new net A7: J?.3 (Pin_3)
- new net A8: J?.12 (Pin_12)
- new net A9: J?.11 (Pin_11)
- new net B0: J?.2 (Pin_2)
- new net B1: J?.1 (Pin_1)
- new net B3: J?.6 (Pin_6)
- new net B4: J?.5 (Pin_5)
- new net B5: J?.4 (Pin_4)
- new net B6: J?.3 (Pin_3)
- new net B7: J?.2 (Pin_2)
- new net SWCLK: J?.3 (Pin_3)
- new net SWDIO: J?.4 (Pin_4)
Other:
- note added: "Power Supply 3.3V 300mA"

Commit message: create GPIO Pins
Parts:
- removed FB?: Ferrite_Bead, symbol Device:Ferrite_Bead
- C1: footprint (none) -> Capacitor_Tantalum_SMD:CP_EIA-3216-10_Kemet-I_Pad1.58x1.35mm_HandSolder
- C10, C4, C5, C6, C7, C8, C9: renamed from C?; footprint (none) -> Capacitor_SMD:C_0805_2012Metric_Pad1.18x1.45mm_HandSolder
- C2, C3: footprint (none) -> Capacitor_SMD:C_0805_2012Metric_Pad1.18x1.45mm_HandSolder
- D1: footprint (none) -> Diode_SMD:D_SOD-123
- D2: footprint (none) -> LED_SMD:LED_0805_2012Metric_Pad1.15x1.40mm_HandSolder
- J1, J3: renamed from J?; footprint (none) -> Connector_PinSocket_2.54mm:PinSocket_1x12_P2.54mm_Vertical
- J2: renamed from J?; footprint (none) -> Connector_PinSocket_2.54mm:PinSocket_1x04_P2.54mm_Vertical
- R1: footprint (none) -> Resistor_SMD:R_0805_2012Metric_Pad1.20x1.40mm_HandSolder
- SW1: renamed from SW?; footprint (none) -> Button_Switch_THT:SW_PUSH_6mm
- U1: footprint (none) -> Package_QFP:LQFP-32_7x7mm_P0.8mm
- U2: footprint Package_TO_SOT_SMD:SOT-223-3_TabPin2 -> Package_TO_SOT_SMD:SOT-23-5_HandSoldering
- Y1: renamed from Y?; footprint (none) -> Crystal:Crystal_Round_D3.0mm_Vertical
Connections:
- net +3V3: now also C6.1, C8.1, U1.5 (VDDA)
- net A0: now also U1.6 (A0)
- net A1: now also U1.7 (A1)
- net A10: now also U1.20 (PA10)
- net A11: now also U1.21 (PA11)
- net A12: now also U1.22 (PA12)
- net A15: now also U1.25 (PA15)
- net A2: now also U1.8 (A2)
- net A3: now also U1.9 (A3)
- net A4: now also U1.10 (A4)
- net A5: now also U1.11 (A5)
- net A6: now also U1.12 (A6)
- net A7: now also U1.13 (A7)
- net A8: now also U1.18 (PA8)
- net A9: now also U1.19 (PA9)
- net B0: now also U1.14 (B0)
- net B1: now also U1.15 (B1)
- net B3: now also U1.26 (PB3)
- net B4: now also U1.27 (PB4)
- net B5: now also U1.28 (PB5)
- net B6: now also U1.29 (PB6)
- net B7: now also U1.30 (PB7)
- net SWCLK: now also U1.24 (PA14)
- net SWDIO: now also U1.23 (PA13)
Other:
- moved on the sheet: J1, J3
